File: PCB/SofleKeyboard.sch (KiCad schematic (older format))
At the start: 85 parts, among them J1 LED, J2 4PIN, J3 OLED, P1 i2c_pin, P2 i2c_pin, SW1 SW_PUSH, SW10 SW_PUSH, SW11 SW_PUSH, SW12 SW_PUSH, SW13 SW_PUSH, SW14 SW_PUSH, SW15 SW_PUSH, SW16 SW_PUSH, SW17 SW_PUSH, SW18 SW_PUSH, SW19 SW_PUSH, SW2 SW_PUSH, SW20 SW_PUSH, SW21 SW_PUSH, SW22 SW_PUSH, SW23 SW_PUSH, SW24 SW_PUSH, SW25 Rotary_Encoder_Switch, SW26 SW_PUSH, SW27 SW_PUSH, SW28 SW_PUSH, SW29 SW_PUSH, SW3 SW_PUSH, SW30 SW_PUSH, SW4 SW_PUSH, SW5 SW_PUSH, SW6 SW_PUSH, SW7 SW_PUSH, SW8 SW_PUSH, SW9 SW_PUSH, U1 ProMicro

Commit message: Add name to the PCB
Parts:
- J2: footprint SofleKeyboard-footprint:MJ-4PP-9_rev3 -> SofleKeyboard-footprint:MJ-4PP-9
- U1: footprint SofleKeyboard-footprint:ProMicro_rev2 -> SofleKeyboard-footprint:ProMicro
Changed lines of the file:
@@
 F 0 "U1" H 3200 3350 60  0000 C CNN
 F 1 "ProMicro" H 3200 1950 60  0000 C CNN
-F 2 "SofleKeyboard-footprint:ProMicro_rev2" H 3300 1600 60  0001 C CNN
+F 2 "SofleKeyboard-footprint:ProMicro" H 3300 1600 60  0001 C CNN
 F 3 "" H 3300 1600 60  0000 C CNN
 	1    3200 2650
@@
 F 0 "J2" H 2650 4650 60  0000 C CNN
 F 1 "4PIN" H 2650 4050 60  0000 C CNN
-F 2 "SofleKeyboard-footprint:MJ-4PP-9_rev3" H 2700 4300 60  0001 C CNN
+F 2 "SofleKeyboard-footprint:MJ-4PP-9" H 2700 4300 60  0001 C CNN
 F 3 "" H 2700 4300 60  0000 C CNN
 	1    2700 4350

Commit message: Add footprints for MX only socketed switches. Use those switches on the board
Parts:
- SW1, SW10, SW11, SW12, SW13, SW14, SW15, SW16, SW17, SW18, SW19, SW2, SW20, SW21, SW22, SW23, SW24, SW27, SW28, SW29, SW3, SW30, SW4, SW5, SW6, SW7, SW8, SW9: footprint SofleKeyboard-footprint:CherryMX_KailhLowProfile_Hotswap -> SofleKeyboard-footprint:CherryMX_Hotswap
- SW26: footprint SofleKeyboard-footprint:CherryMX_KailhLowProfile_Hotswap_1.5 -> SofleKeyboard-footprint:CherryMX_Hotswap_1.5
Changed lines of the file:
@@
 EESchema Schematic File Version 4
-LIBS:SofleKeyboard-cache
 EELAYER 30 0
 EELAYER END
@@
 F 0 "SW26" H 6600 5000 50  0000 C CNN
 F 1 "SW_PUSH" H 6600 4750 50  0000 C CNN
-F 2 "SofleKeyboard-footprint:CherryMX_KailhLowProfile_Hotswap_1.5" H 6600 4850 50  0001 C CNN
+F 2 "SofleKeyboard-footprint:CherryMX_Hotswap_1.5" H 6600 4850 50  0001 C CNN
 F 3 "" H 6600 4850 50  0000 C CNN
 	1    6600 4850
@@
 F 0 "SW1" H 5800 2400 50  0000 C CNN
 F 1 "SW_PUSH" H 5800 2150 50  0000 C CNN
-F 2 "SofleKeyboard-footprint:CherryMX_KailhLowProfile_Hotswap" H 5800 2250 50  0001 C CNN
+F 2 "SofleKeyboard-footprint:CherryMX_Hotswap" H 5800 2250 50  0001 C CNN
 F 3 "" H 5800 2250 50  0000 C CNN
 	1    5800 2250
@@
 F 0 "SW2" H 6600 2400 50  0000 C CNN
 F 1 "SW_PUSH" H 6600 2150 50  0000 C CNN
-F 2 "SofleKeyboard-footprint:CherryMX_KailhLowProfile_Hotswap" H 6600 2250 50  0001 C CNN
+F 2 "SofleKeyboard-footprint:CherryMX_Hotswap" H 6600 2250 50  0001 C CNN
 F 3 "" H 6600 2250 50  0000 C CNN
 	1    6600 2250
@@
 F 0 "SW3" H 7400 2400 50  0000 C CNN
 F 1 "SW_PUSH" H 7400 2150 50  0000 C CNN
-F 2 "SofleKeyboard-footprint:CherryMX_KailhLowProfile_Hotswap" H 7400 2250 50  0001 C CNN
+F 2 "SofleKeyboard-footprint:CherryMX_Hotswap" H 7400 2250 50  0001 C CNN
 F 3 "" H 7400 2250 50  0000 C CNN
 	1    7400 2250
@@
 F 0 "SW4" H 8200 2400 50  0000 C CNN
 F 1 "SW_PUSH" H 8200 2150 50  0000 C CNN
-F 2 "SofleKeyboard-footprint:CherryMX_KailhLowProfile_Hotswap" H 8200 2250 50  0001 C CNN
+F 2 "SofleKeyboard-footprint:CherryMX_Hotswap" H 8200 2250 50  0001 C CNN
 F 3 "" H 8200 2250 50  0000 C CNN
 	1    8200 2250
@@
 F 0 "SW5" H 9000 2400 50  0000 C CNN
 F 1 "SW_PUSH" H 9000 2150 50  0000 C CNN
-F 2 "SofleKeyboard-footprint:CherryMX_KailhLowProfile_Hotswap" H 9000 2250 50  0001 C CNN
+F 2 "SofleKeyboard-footprint:CherryMX_Hotswap" H 9000 2250 50  0001 C CNN
 F 3 "" H 9000 2250 50  0000 C CNN
 	1    9000 2250
@@
 F 0 "SW6" H 9800 2400 50  0000 C CNN
 F 1 "SW_PUSH" H 9800 2200 50  0000 C CNN
-F 2 "SofleKeyboard-footprint:CherryMX_KailhLowProfile_Hotswap" H 9800 2250 50  0001 C CNN
+F 2 "SofleKeyboard-footprint:CherryMX_Hotswap" H 9800 2250 50  0001 C CNN
 F 3 "" H 9800 2250 50  0000 C CNN
 	1    9800 2250
@@
 F 0 "SW8" H 6600 3050 50  0000 C CNN
 F 1 "SW_PUSH" H 6600 2800 50  0000 C CNN
-F 2 "SofleKeyboard-footprint:CherryMX_KailhLowProfile_Hotswap" H 6600 2900 50  0001 C CNN
+F 2 "SofleKeyboard-footprint:CherryMX_Hotswap" H 6600 2900 50  0001 C CNN
 F 3 "" H 6600 2900 50  0000 C CNN
 	1    6600 2900
@@
 F 0 "SW9" H 7400 3050 50  0000 C CNN
 F 1 "SW_PUSH" H 7400 2800 50  0000 C CNN
-F 2 "SofleKeyboard-footprint:CherryMX_KailhLowProfile_Hotswap" H 7400 2900 50  0001 C CNN
+F 2 "SofleKeyboard-footprint:CherryMX_Hotswap" H 7400 2900 50  0001 C CNN
 F 3 "" H 7400 2900 50  0000 C CNN
 	1    7400 2900
@@
 F 0 "SW10" H 8200 3050 50  0000 C CNN
 F 1 "SW_PUSH" H 8200 2800 50  0000 C CNN
-F 2 "SofleKeyboard-footprint:CherryMX_KailhLowProfile_Hotswap" H 8200 2900 50  0001 C CNN
+F 2 "SofleKeyboard-footprint:CherryMX_Hotswap" H 8200 2900 50  0001 C CNN
 F 3 "" H 8200 2900 50  0000 C CNN
 	1    8200 2900
@@
 F 0 "SW11" H 9000 3050 50  0000 C CNN
 F 1 "SW_PUSH" H 9000 2800 50  0000 C CNN
-F 2 "SofleKeyboard-footprint:CherryMX_KailhLowProfile_Hotswap" H 9000 2900 50  0001 C CNN
+F 2 "SofleKeyboard-footprint:CherryMX_Hotswap" H 9000 2900 50  0001 C CNN
 F 3 "" H 9000 2900 50  0000 C CNN
 	1    9000 2900
@@
 F 0 "SW12" H 9800 3050 50  0000 C CNN
 F 1 "SW_PUSH" H 9800 2800 50  0000 C CNN
-F 2 "SofleKeyboard-footprint:CherryMX_KailhLowProfile_Hotswap" H 9800 2900 50  0001 C CNN
+F 2 "SofleKeyboard-footprint:CherryMX_Hotswap" H 9800 2900 50  0001 C CNN
 F 3 "" H 9800 2900 50  0000 C CNN
 	1    9800 2900
@@
 F 0 "SW7" H 5800 3050 50  0000 C CNN
 F 1 "SW_PUSH" H 5800 2800 50  0000 C CNN
-F 2 "SofleKeyboard-footprint:CherryMX_KailhLowProfile_Hotswap" H 5800 2900 50  0001 C CNN
+F 2 "SofleKeyboard-footprint:CherryMX_Hotswap" H 5800 2900 50  0001 C CNN
 F 3 "" H 5800 2900 50  0000 C CNN
 	1    5800 2900
@@
 F 0 "SW13" H 5800 3700 50  0000 C CNN
 F 1 "SW_PUSH" H 5800 3450 50  0000 C CNN
-F 2 "SofleKeyboard-footprint:CherryMX_KailhLowProfile_Hotswap" H 5800 3550 50  0001 C CNN
+F 2 "SofleKeyboard-footprint:CherryMX_Hotswap" H 5800 3550 50  0001 C CNN
 F 3 "" H 5800 3550 50  0000 C CNN
 	1    5800 3550
@@
 F 0 "SW14" H 6600 3700 50  0000 C CNN
 F 1 "SW_PUSH" H 6600 3450 50  0000 C CNN
-F 2 "SofleKeyboard-footprint:CherryMX_KailhLowProfile_Hotswap" H 6600 3550 50  0001 C CNN
+F 2 "SofleKeyboard-footprint:CherryMX_Hotswap" H 6600 3550 50  0001 C CNN
 F 3 "" H 6600 3550 50  0000 C CNN
 	1    6600 3550
@@
 F 0 "SW15" H 7400 3700 50  0000 C CNN
 F 1 "SW_PUSH" H 7400 3450 50  0000 C CNN
-F 2 "SofleKeyboard-footprint:CherryMX_KailhLowProfile_Hotswap" H 7400 3550 50  0001 C CNN
+F 2 "SofleKeyboard-footprint:CherryMX_Hotswap" H 7400 3550 50  0001 C CNN
 F 3 "" H 7400 3550 50  0000 C CNN
 	1    7400 3550
@@
 F 0 "SW16" H 8200 3700 50  0000 C CNN
 F 1 "SW_PUSH" H 8200 3450 50  0000 C CNN
-F 2 "SofleKeyboard-footprint:CherryMX_KailhLowProfile_Hotswap" H 8200 3550 50  0001 C CNN
+F 2 "SofleKeyboard-footprint:CherryMX_Hotswap" H 8200 3550 50  0001 C CNN
 F 3 "" H 8200 3550 50  0000 C CNN
 	1    8200 3550
@@
 F 0 "SW17" H 9000 3700 50  0000 C CNN
 F 1 "SW_PUSH" H 9000 3450 50  0000 C CNN
-F 2 "SofleKeyboard-footprint:CherryMX_KailhLowProfile_Hotswap" H 9000 3550 50  0001 C CNN
+F 2 "SofleKeyboard-footprint:CherryMX_Hotswap" H 9000 3550 50  0001 C CNN
 F 3 "" H 9000 3550 50  0000 C CNN
 	1    9000 3550
@@
 F 0 "SW18" H 9800 3700 50  0000 C CNN
 F 1 "SW_PUSH" H 9800 3450 50  0000 C CNN
-F 2 "SofleKeyboard-footprint:CherryMX_KailhLowProfile_Hotswap" H 9800 3550 50  0001 C CNN
+F 2 "SofleKeyboard-footprint:CherryMX_Hotswap" H 9800 3550 50  0001 C CNN
 F 3 "" H 9800 3550 50  0000 C CNN
 	1    9800 3550
@@
 F 0 "SW21" H 7400 4350 50  0000 C CNN
 F 1 "SW_PUSH" H 7400 4100 50  0000 C CNN
-F 2 "SofleKeyboard-footprint:CherryMX_KailhLowProfile_Hotswap" H 7400 4200 50  0001 C CNN
+F 2 "SofleKeyboard-footprint:CherryMX_Hotswap" H 7400 4200 50  0001 C CNN
 F 3 "" H 7400 4200 50  0000 C CNN
 	1    7400 4200
@@
 F 0 "SW22" H 8200 4350 50  0000 C CNN
 F 1 "SW_PUSH" H 8200 4100 50  0000 C CNN
-F 2 "SofleKeyboard-footprint:CherryMX_KailhLowProfile_Hotswap" H 8200 4200 50  0001 C CNN
+F 2 "SofleKeyboard-footprint:CherryMX_Hotswap" H 8200 4200 50  0001 C CNN
 F 3 "" H 8200 4200 50  0000 C CNN
 	1    8200 4200
@@
 F 0 "SW23" H 9000 4350 50  0000 C CNN
 F 1 "SW_PUSH" H 9000 4100 50  0000 C CNN
-F 2 "SofleKeyboard-footprint:CherryMX_KailhLowProfile_Hotswap" H 9000 4200 50  0001 C CNN
+F 2 "SofleKeyboard-footprint:CherryMX_Hotswap" H 9000 4200 50  0001 C CNN
 F 3 "" H 9000 4200 50  0000 C CNN
 	1    9000 4200
@@
 F 0 "SW24" H 9800 4350 50  0000 C CNN
 F 1 "SW_PUSH" H 9800 4100 50  0000 C CNN
-F 2 "SofleKeyboard-footprint:CherryMX_KailhLowProfile_Hotswap" H 9800 4200 50  0001 C CNN
+F 2 "SofleKeyboard-footprint:CherryMX_Hotswap" H 9800 4200 50  0001 C CNN
 F 3 "" H 9800 4200 50  0000 C CNN
 	1    9800 4200
@@
 F 0 "SW20" H 6600 4350 50  0000 C CNN
 F 1 "SW_PUSH" H 6600 4100 50  0000 C CNN
-F 2 "SofleKeyboard-footprint:CherryMX_KailhLowProfile_Hotswap" H 6600 4200 50  0001 C CNN
+F 2 "SofleKeyboard-footprint:CherryMX_Hotswap" H 6600 4200 50  0001 C CNN
 F 3 "" H 6600 4200 50  0000 C CNN
 	1    6600 4200
@@
 F 0 "SW19" H 5800 4350 50  0000 C CNN
 F 1 "SW_PUSH" H 5800 4100 50  0000 C CNN
-F 2 "SofleKeyboard-footprint:CherryMX_KailhLowProfile_Hotswap" H 5800 4200 50  0001 C CNN
+F 2 "SofleKeyboard-footprint:CherryMX_Hotswap" H 5800 4200 50  0001 C CNN
 F 3 "" H 5800 4200 50  0000 C CNN
 	1    5800 4200
@@
 F 0 "SW27" H 7400 5000 50  0000 C CNN
 F 1 "SW_PUSH" H 7400 4750 50  0000 C CNN
-F 2 "SofleKeyboard-footprint:CherryMX_KailhLowProfile_Hotswap" H 7400 4850 50  0001 C CNN
+F 2 "SofleKeyboard-footprint:CherryMX_Hotswap" H 7400 4850 50  0001 C CNN
 F 3 "" H 7400 4850 50  0000 C CNN
 	1    7400 4850
@@
 F 0 "SW28" H 8200 5000 50  0000 C CNN
 F 1 "SW_PUSH" H 8200 4750 50  0000 C CNN
-F 2 "SofleKeyboard-footprint:CherryMX_KailhLowProfile_Hotswap" H 8200 4850 50  0001 C CNN
+F 2 "SofleKeyboard-footprint:CherryMX_Hotswap" H 8200 4850 50  0001 C CNN
 F 3 "" H 8200 4850 50  0000 C CNN
 	1    8200 4850
@@
 F 0 "SW29" H 9000 5000 50  0000 C CNN
 F 1 "SW_PUSH" H 9000 4750 50  0000 C CNN
-F 2 "SofleKeyboard-footprint:CherryMX_KailhLowProfile_Hotswap" H 9000 4850 50  0001 C CNN
+F 2 "SofleKeyboard-footprint:CherryMX_Hotswap" H 9000 4850 50  0001 C CNN
 F 3 "" H 9000 4850 50  0000 C CNN
 	1    9000 4850
@@
 F 0 "SW30" H 9800 5000 50  0000 C CNN
 F 1 "SW_PUSH" H 9800 4750 50  0000 C CNN
-F 2 "SofleKeyboard-footprint:CherryMX_KailhLowProfile_Hotswap" H 9800 4850 50  0001 C CNN
+F 2 "SofleKeyboard-footprint:CherryMX_Hotswap" H 9800 4850 50  0001 C CNN
 F 3 "" H 9800 4850 50  0000 C CNN
 	1    9800 4850

Commit message: WIP routing micro
Parts:
- removed P1, P2: i2c_pin, SofleKeyboard-footprint:1pin_conn, symbol SofleKeyboard-rescue:i2c_pin-Lily58-cache-Lily58_Pro-rescue
- removed W1: jumper, SofleKeyboard-footprint:jumper_data, symbol Device:Jumper
- added JP10: IC2SDA, Jumper:SolderJumper-2_P1.3mm_Open_TrianglePad1.0x1.5mm, symbol Device:Jumper_NO_Small
- added JP11: Serial, Jumper:SolderJumper-2_P1.3mm_Bridged2Bar_Pad1.0x1.5mm, symbol Device:Jumper_NC_Small
- added JP9: I2CSCL, Jumper:SolderJumper-2_P1.3mm_Open_TrianglePad1.0x1.5mm, symbol Device:Jumper_NO_Small
- R1, R2: footprint SofleKeyboard-footprint:RESISTOR_mini -> SofleKeyboard-footprint:R_1206_DoubleSided
- U1: footprint SofleKeyboard-footprint:ProMicro -> Keebio:ArduinoProMicro-ZigZag
Connections:
- net DATA: now also JP11.1
- net SCL: now also JP9.1
- net SDA: now also JP10.2
- net i2c_c: now also JP9.2
- net i2c_d: now also JP10.1, JP11.2
Changed lines of the file:
@@
 F 0 "U1" H 3200 3350 60  0000 C CNN
 F 1 "ProMicro" H 3200 1950 60  0000 C CNN
-F 2 "SofleKeyboard-footprint:ProMicro" H 3300 1600 60  0001 C CNN
+F 2 "Keebio:ArduinoProMicro-ZigZag" H 3300 1600 60  0001 C CNN
 F 3 "" H 3300 1600 60  0000 C CNN
 	1    3200 2650
@@
 F 0 "R1" V 4500 4950 50  0000 C BNN
 F 1 "R" V 4400 4950 50  0000 C CNN
-F 2 "SofleKeyboard-footprint:RESISTOR_mini" V 4330 4950 50  0001 C CNN
+F 2 "SofleKeyboard-footprint:R_1206_DoubleSided" V 4330 4950 50  0001 C CNN
 F 3 "" H 4400 4950 50  0001 C CNN
 	1    4400 4950
@@
 F 0 "R2" V 4650 4950 50  0000 C BNN
 F 1 "R" V 4550 4950 50  0000 C CNN
-F 2 "SofleKeyboard-footprint:RESISTOR_mini" V 4480 4950 50  0001 C CNN
+F 2 "SofleKeyboard-footprint:R_1206_DoubleSided" V 4480 4950 50  0001 C CNN
 F 3 "" H 4550 4950 50  0001 C CNN
 	1    4550 4950
@@
 Wire Wire Line
 	3150 4450 3250 4450
-$Comp
-L SofleKeyboard-rescue:i2c_pin-Lily58-cache-Lily58_Pro-rescue P1
-U 1 1 5B8F6780
-P 3550 4000
-F 0 "P1" H 3550 4100 50  0000 C CNN
-F 1 "i2c_pin" V 3650 4000 50  0000 C CNN
-F 2 "SofleKeyboard-footprint:1pin_conn" H 3550 4000 50  0001 C CNN
-F 3 "" H 3550 4000 50  0001 C CNN
-	1    3550 4000
-	0    -1   -1   0
-$EndComp
-$Comp
-L SofleKeyboard-rescue:i2c_pin-Lily58-cache-Lily58_Pro-rescue P2
-U 1 1 5B8F6980
-P 3550 4750
-F 0 "P2" H 3550 4650 50  0000 C CNN
-F 1 "i2c_pin" V 3650 4750 50  0000 C CNN
-F 2 "SofleKeyboard-footprint:1pin_conn" H 3550 4750 50  0001 C CNN
-F 3 "" H 3550 4750 50  0001 C CNN
-	1    3550 4750
-	0    1    1    0
-$EndComp
-Wire Wire Line
-	3150 4550 3550 4550
-Wire Wire Line
-	3150 4200 3550 4200
 Wire Wire Line
 	3250 4150 3250 4350
 Wire Wire Line
 	3250 4450 3250 4600
-$Comp
-L Device:Jumper W1
-U 1 1 5B900157
-P 3850 4550
-F 0 "W1" H 3850 4500 50  0000 C CNN
-F 1 "jumper" H 3850 4700 50  0000 C CNN
-F 2 "SofleKeyboard-footprint:jumper_data" H 3850 4550 50  0001 C CNN
-F 3 "" H 3850 4550 50  0000 C CNN
-	1    3850 4550
-	-1   0    0    1
-$EndComp
 Text GLabel 2550 2200 0    50   Input ~ 0
 DATA
-Text GLabel 4150 4550 2    50   Input ~ 0
+Text GLabel 3650 4300 2    50   Input ~ 0
 DATA
 $Comp
@@
 Wire Wire Line
 	3850 2400 4150 2400
-Connection ~ 3550 4550
 $Comp
 L SofleKeyboard-rescue:SW_PUSH-Lily58-cache-Lily58_Pro-rescue SW30
@@
 Text Label 3300 4200 0    50   ~ 0
 i2c_c
+$Comp
+L Device:Jumper_NO_Small JP9
+U 1 1 5E98AECB
+P 3600 4100
+F 0 "JP9" V 3554 4148 50  0000 L CNN
+F 1 "I2CSCL" V 3650 4150 50  0000 L CNN
+F 2 "Jumper:SolderJumper-2_P1.3mm_Open_TrianglePad1.0x1.5mm" H 3600 4100 50  0001 C CNN
+F 3 "~" H 3600 4100 50  0001 C CNN
+	1    3600 4100
+	0    1    1    0
+$EndComp
+Wire Wire Line
+	3150 4200 3600 4200
+Text GLabel 3700 4850 2    50   Input ~ 0
+SDA
+Text GLabel 3650 3850 2    50   Input ~ 0
+SCL
+Wire Wire Line
+	3600 3850 3600 4000
+$Comp
+L Device:Jumper_NO_Small JP10
+U 1 1 5E9C09A0
+P 3600 4650
+F 0 "JP10" V 3554 4698 50  0000 L CNN
+F 1 "IC2SDA" V 3645 4698 50  0000 L CNN
+F 2 "Jumper:SolderJumper-2_P1.3mm_Open_TrianglePad1.0x1.5mm" H 3600 4650 50  0001 C CNN
+F 3 "~" H 3600 4650 50  0001 C CNN
+	1    3600 4650
+	0    1    1    0
+$EndComp
+Wire Wire Line
+	3150 4550 3600 4550
+Wire Wire Line
+	3600 4750 3600 4850
+$Comp
+L Device:Jumper_NC_Small JP11
+U 1 1 5E9D186B
+P 3600 4450
+F 0 "JP11" V 3554 4525 50  0000 L CNN
+F 1 "Serial" V 3645 4525 50  0000 L CNN
+F 2 "Jumper:SolderJumper-2_P1.3mm_Bridged2Bar_Pad1.0x1.5mm" H 3600 4450 50  0001 C CNN
+F 3 "~" H 3600 4450 50  0001 C CNN
+	1    3600 4450
+	0    1    1    0
+$EndComp
+Connection ~ 3600 4550
+Wire Wire Line
+	3600 4350 3600 4300
+Wire Wire Line
+	3600 4300 3650 4300
+Wire Wire Line
+	3600 3850 3650 3850
+Wire Wire Line
+	3600 4850 3700 4850
 $EndSCHEMATC

Commit message: Adding 3d models
Parts:
- U1: footprint Keebio:ArduinoProMicro-ZigZag -> SofleKeyboard-footprint:ArduinoProMicro-ZigZag-DoubleSided
Changed lines of the file:
@@
 F 0 "U1" H 3200 3350 60  0000 C CNN
 F 1 "ProMicro" H 3200 1950 60  0000 C CNN
-F 2 "Keebio:ArduinoProMicro-ZigZag" H 3300 1600 60  0001 C CNN
+F 2 "SofleKeyboard-footprint:ArduinoProMicro-ZigZag-DoubleSided" H 3300 1600 60  0001 C CNN
 F 3 "" H 3300 1600 60  0000 C CNN
 	1    3200 2650

Commit message: WIP shape
Parts:
- RSW1: footprint SofleKeyboard-footprint:TACT_SWITCH_TVBP06 -> Button_Switch_SMD:SW_SPST_B3U-3000P-B
Changed lines of the file:
@@
 F 0 "RSW1" H 2500 3956 40  0000 C CNN
 F 1 "SW_RST" H 2500 3873 50  0000 C CNN
-F 2 "SofleKeyboard-footprint:TACT_SWITCH_TVBP06" H 2500 3700 50  0001 C CNN
+F 2 "Button_Switch_SMD:SW_SPST_B3U-3000P-B" H 2500 3700 50  0001 C CNN
 F 3 "" H 2500 3700 50  0001 C CNN
 	1    2500 3700

Commit message: WIP - moving things more around
Parts:
- RSW1: footprint Button_Switch_SMD:SW_SPST_B3U-3000P-B -> SofleKeyboard-footprint:TACT_SWITCH_TVBP06
Changed lines of the file:
@@
 F 0 "RSW1" H 2500 3956 40  0000 C CNN
 F 1 "SW_RST" H 2500 3873 50  0000 C CNN
-F 2 "Button_Switch_SMD:SW_SPST_B3U-3000P-B" H 2500 3700 50  0001 C CNN
+F 2 "SofleKeyboard-footprint:TACT_SWITCH_TVBP06" H 2500 3700 50  0001 C CNN
 F 3 "" H 2500 3700 50  0001 C CNN
 	1    2500 3700
