File: Sofle_Choc_v2/Case/PCBTop/SofleKeyboardTopPlate.kicad_pcb (KiCad board)
At the start: 2 copper layers, 143.4 x 111.8 mm, 34 parts, among them SW2 KEY_SWITCH

Commit message: Bump to version 2.1
Other:
- board text added: "Sofle Choc v2.1, Brian Low"
- board text removed: "Sofle Choc v2.0, Brian Low"
