File: Sofle_v2.0w/PCB/sofle_left/SofleKeyboard.kicad_pcb (KiCad board)
At the start: 2 copper layers, 143.5 x 115.5 mm, 74 parts, among them J1 OLED, J2 LED, SW1 SW_PUSH, SW10 SW_PUSH, SW11 SW_PUSH, SW12 SW_PUSH, SW13 SW_PUSH, SW14 SW_PUSH, SW15 SW_PUSH, SW16 SW_PUSH, SW17 SW_PUSH, SW18 SW_PUSH, SW19 SW_PUSH, SW2 SW_PUSH, SW20 SW_PUSH, SW21 SW_PUSH, SW22 SW_PUSH, SW23 SW_PUSH, SW24 SW_PUSH, SW25 Rotary_Encoder_Switch, SW26 SW_PUSH, SW27 SW_PUSH, SW28 SW_PUSH, SW29 SW_PUSH, SW3 SW_PUSH, SW30 SW_PUSH, SW4 SW_PUSH, SW5 SW_PUSH, SW6 SW_PUSH, SW7 SW_PUSH, SW8 SW_PUSH, SW9 SW_PUSH, U1 ProMicro

Commit message: I fit both pcbs in and routed a little
Parts:
- removed SW26: SW_PUSH, SofleKeyboard-footprint:CherryMX_KailhLowProfile_Hotswap_OneSide_1.5
- removed SW27: SW_PUSH, SofleKeyboard-footprint:CherryMX_KailhLowProfile_Hotswap_OneSide
- added SW110: SW_PUSH, SofleKeyboard-footprint:CherryMX_KailhLowProfile_Hotswap_OneSide_1.5, F.Cu at (215.5, 133.4)
- added SW115: SW_PUSH, SofleKeyboard-footprint:CherryMX_KailhLowProfile_Hotswap_OneSide, F.Cu at (194.6, 128.4)
- renumbered BATJ1 to BATJ101, BATJ2 to BATJ102, D1 to D101, D7 to D102, D13 to D103, D19 to D104, D25 to D105, D2 to D106, D8 to D107, D14 to D108, D20 to D109, D26 to D110, D3 to D111, D9 to D112, D15 to D113, D21 to D114, D27 to D115, D4 to D116, D10 to D117, D16 to D118, D22 to D119, D28 to D120, D5 to D121, D11 to D122, D17 to D123, D23 to D124, D29 to D125, D6 to D126, D12 to D127, D18 to D128, D24 to D129, D30 to D130, J1 to J101, J2 to J102, PSW1 to PSW101, RSW1 to RSW101, SW25 to SW101, SW1 to SW102, SW7 to SW103, SW13 to SW104, SW19 to SW105, SW2 to SW106, SW8 to SW107, SW14 to SW108, SW20 to SW109, SW3 to SW111, SW9 to SW112, SW15 to SW113, SW21 to SW114, SW4 to SW116, SW10 to SW117, SW16 to SW118, SW22 to SW119, SW28 to SW120, SW5 to SW121, SW11 to SW122, SW17 to SW123, SW23 to SW124, SW29 to SW125, SW6 to SW126, SW12 to SW127, SW18 to SW128, SW24 to SW129, SW30 to SW130, TH7 to TH101, TH6 to TH102, TH5 to TH103, TH4 to TH104, TH3 to TH105, TH2 to TH106, TH1 to TH107, U1 to U101
